File: Drivers.sch (KiCad schematic (older format))
At the start: 12 parts

Commit message: added gate drivers, increased FET spacing
Parts:
- added R304, R305, R306, R307, R308, R309: R, Resistors_SMD:R_1812, symbol R
- added R310, R311, R312: R, Resistors_SMD:R_0603, symbol R
- added U301, U302, U303, U304, U305, U306: 1EDI60H12AH, VFD_parts:PG-DSO-8-59, symbol 1EDI60H12AH
- renumbered C4 to C301, C1 to C302, C5 to C303, C2 to C304, C6 to C305, C3 to C306, D7 to D301, D8 to D302, D9 to D303, R1 to R301, R2 to R302, R3 to R303
Connections:
- net labels added: GNDD, Q1L_DS, Q1L_G, Q2L_DS, Q2L_G, Q3L_DS, Q3L_G, VCC
- wire segments 24 -> 84
Other:
- note added: "The Eice Driver has a neat inverting pin behaviour\nShown here wired to prohibit shoot-through\nNot the final gate logic."
- moved on the sheet: C301, D301
